File: pwm/esp-pcb/esp-pwm.sch (KiCad schematic (older format))
At the start: 14 parts, among them Q1 2N3904, Q2 2N3904, Q3 IRF540N, SW1 SW_Push, SW2 SW_Push, U1 LM1117-3.3, U2 ESP-12E

Commit message: Created PWM2
Parts:
- SW1: value SW_Push -> RST
- SW2: value SW_Push -> FLASH
Changed lines of the file:
@@
 EESchema Schematic File Version 4
+LIBS:esp-pwm-cache
 EELAYER 26 0
 EELAYER END
@@
 P 7400 2650
 F 0 "SW2" H 7400 2935 50  0000 C CNN
-F 1 "SW_Push" H 7400 2844 50  0000 C CNN
+F 1 "FLASH" H 7400 2844 50  0000 C CNN
 F 2 "" H 7400 2850 50  0001 C CNN
 F 3 "" H 7400 2850 50  0001 C CNN
@@
 P 4600 2650
 F 0 "SW1" H 4600 2935 50  0000 C CNN
-F 1 "SW_Push" H 4600 2844 50  0000 C CNN
+F 1 "RST" H 4600 2844 50  0000 C CNN
 F 2 "" H 4600 2850 50  0001 C CNN
 F 3 "" H 4600 2850 50  0001 C CNN
