File: pwm-2/esp-pcb/esp-pwm.kicad_pcb (KiCad board)
At the start: 2 copper layers, 25 parts, among them J1 Screw_Terminal_01x02, J2 Conn_01x03_Male, J3 Screw_Terminal_01x02, J4 Screw_Terminal_01x02, Q1 2N3904, Q2 2N3904, Q3 IRF540N, Q4 2N3904, Q5 2N3904, Q6 IRF540N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

Commit message: PWM2
Parts:
- C1: footprint Capacitor_THT:CP_Radial_D4.0mm_P2.00mm -> Capacitor_THT:C_Disc_D7.5mm_W2.5mm_P5.00mm
- C2: footprint Capacitor_THT:C_Disc_D3.0mm_W1.6mm_P2.50mm -> Capacitor_THT:CP_Radial_D5.0mm_P2.50mm
- J2: footprint Connector_PinHeader_1.00mm:PinHeader_1x03_P1.00mm_Vertical -> Connector_PinHeader_2.54mm:PinHeader_1x03_P2.54mm_Horizontal
- Q1, Q2, Q4, Q5: footprint Package_TO_SOT_THT:TO-92_Inline -> Package_TO_SOT_THT:TO-92_Inline_Wide
- R10, R5, R6, R7, R8, R9: footprint Resistor_THT:R_Axial_DIN0207_L6.3mm_D2.5mm_P2.54mm_Vertical -> Resistor_THT:R_Axial_DIN0204_L3.6mm_D1.6mm_P7.62mm_Horizontal
- R4: footprint Resistor_THT:R_Axial_DIN0207_L6.3mm_D2.5mm_P2.54mm_Vertical -> Resistor_THT:R_Axial_DIN0207_L6.3mm_D2.5mm_P7.62mm_Horizontal
- U2: moved to B.Cu
- moved J1 101.8 mm to (205.7, 45.7), turned to 270 degrees
- moved U1 95.6 mm to (205.7, 61.0), turned to 270 degrees
- moved C2 86.1 mm to (205.7, 73.7), turned to 180 degrees
- moved C1 84.5 mm to (205.7, 55.9), turned to 180 degrees
- moved R2 81.2 mm to (195.6, 61.0), turned to 90 degrees
- moved R6 80.1 mm to (190.5, 38.1), turned to 270 degrees
- moved Q6 79.8 mm to (203.2, 96.5), turned to 180 degrees
- moved R1 72.7 mm to (195.6, 66.0), turned to 270 degrees
- moved Q1 72.2 mm to (198.1, 50.8), turned to 90 degrees
- moved R8 68.4 mm to (200.7, 76.2), turned to 180 degrees
- moved R5 67.3 mm to (193.0, 48.3), turned to 270 degrees
- moved J3 66.2 mm to (172.7, 38.1)
- moved J4 65.5 mm to (180.3, 96.5), turned to 180 degrees
- moved Q5 64.2 mm to (200.7, 86.4), turned to 180 degrees
- moved R7 62.1 mm to (185.4, 38.1), turned to 270 degrees
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Connections:
- J1 pad 1: Net-(J1-Pad1) -> 12v
- J1 pad 2: Net-(J1-Pad2) -> GND
- J2 pad 1: Net-(J2-Pad1) -> GND
- J2 pad 2: Net-(J2-Pad2) -> RXD
- J2 pad 3: Net-(J2-Pad3) -> TXD
- J3 pad 1: Net-(J3-Pad1) -> 12v
- J3 pad 2: Net-(J3-Pad2) -> OUT1-
- J4 pad 1: Net-(J4-Pad1) -> OUT2-
- J4 pad 2: Net-(J4-Pad2) -> 12v
Routing:
- net 12v: track 0.00 -> 172.7 mm
- net GND: track 7.83 -> 175.4 mm, vias 0 -> 1
- net 3v3: track 7.83 -> 67.7 mm, vias 0 -> 3
- net Net-(R3-Pad2): track 7.12 -> 39.6 mm, vias 0 -> 1
- net OUT2-: track 0.00 -> 30.5 mm
- net OUT1-: track 0.00 -> 30.0 mm
- net CTRL1: track 7.38 -> 32.1 mm, vias 0 -> 1
- net Net-(Q2-Pad3): track 0.00 -> 23.1 mm
- net Net-(Q5-Pad3): track 0.00 -> 20.6 mm, vias 0 -> 2
- net Net-(Q4-Pad3): track 0.00 -> 20.3 mm
- net Net-(Q1-Pad3): track 0.00 -> 15.0 mm
- net Net-(R2-Pad2): track 7.54 -> 16.6 mm, vias 0 -> 1
- net Net-(U2-Pad2): track 7.31 -> 0.00 mm
- net Net-(U2-Pad5): track 7.12 -> 0.00 mm
- net Net-(U2-Pad20): track 7.07 -> 0.00 mm
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