File: pwm-2/esp-pcb/esp-pwm.sch (KiCad schematic (older format))
At the start: 21 parts, among them Q1 2N3904, Q2 2N3904, Q3 IRF540N, Q4 2N3904, Q5 2N3904, Q6 IRF540N, SW2 FLASH, U1 LM1117-3.3, U2 ESP-12E

Commit message: ...
Parts:
- added J1, J3, J4: Screw_Terminal_01x02, TerminalBlock:TerminalBlock_bornier-2_P5.08mm, symbol Connector:Screw_Terminal_01x02
- added J2: Conn_01x03_Male, Connector_PinHeader_1.00mm:PinHeader_1x03_P1.00mm_Vertical, symbol Connector:Conn_01x03_Male
Connections:
- net +12V: now also J1.1 (Pin_1), J3.1 (Pin_1), J4.1 (Pin_1)
- net GND: now also J1.2 (Pin_2), J2.1 (Pin_1)
- net OUT1-: now also J3.2 (Pin_2)
- net OUT2-: now also J4.2 (Pin_2)
- net RXD: now also J2.2 (Pin_2)
- net TXD: now also J2.3 (Pin_3)
Changed lines of the file:
@@
-$EndComp
-$Comp
-L power:+12V #PWR01
-U 1 1 5C31E21D
-P 550 1250
-F 0 "#PWR01" H 550 1100 50  0001 C CNN
-F 1 "+12V" H 565 1423 50  0000 C CNN
-F 2 "" H 550 1250 50  0001 C CNN
-F 3 "" H 550 1250 50  0001 C CNN
-	1    550  1250
-	1    0    0    -1
 $EndComp
 $Comp
@@
 Wire Wire Line
 	9250 2650 9250 2900
-Text GLabel 550  1550 3    50   Input ~ 0
+Text GLabel 850  1250 0    50   Input ~ 0
 12v
 Wire Wire Line
-	550  1250 550  1550
-Text GLabel 850  800  1    50   Input ~ 0
-12v
-Wire Wire Line
 	850  1250 1000 1250
-Wire Wire Line
-	850  800  850  1250
 Text GLabel 9000 1500 1    50   Input ~ 0
 12v
@@
 Wire Wire Line
 	1850 1900 1350 1900
+$Comp
+L Connector:Conn_01x03_Male J2
+U 1 1 5C34B847
+P 7400 700
+F 0 "J2" V 7460 840 50  0000 L CNN
+F 1 "Conn_01x03_Male" V 7551 840 50  0000 L CNN
+F 2 "Connector_PinHeader_1.00mm:PinHeader_1x03_P1.00mm_Vertical" H 7400 700 50  0001 C CNN
+F 3 "~" H 7400 700 50  0001 C CNN
+	1    7400 700
+	0    1    1    0
+$EndComp
+$Comp
+L Connector:Screw_Terminal_01x02 J3
+U 1 1 5C34B967
+P 8050 700
+F 0 "J3" H 8130 692 50  0000 L CNN
+F 1 "Screw_Terminal_01x02" H 8130 601 50  0000 L CNN
+F 2 "TerminalBlock:TerminalBlock_bornier-2_P5.08mm" H 8050 700 50  0001 C CNN
+F 3 "~" H 8050 700 50  0001 C CNN
+	1    8050 700
+	0    -1   -1   0
+$EndComp
+$Comp
+L Connector:Screw_Terminal_01x02 J4
+U 1 1 5C34B9F8
+P 8650 700
+F 0 "J4" H 8730 692 50  0000 L CNN
+F 1 "Screw_Terminal_01x02" H 8730 601 50  0000 L CNN
+F 2 "TerminalBlock:TerminalBlock_bornier-2_P5.08mm" H 8650 700 50  0001 C CNN
+F 3 "~" H 8650 700 50  0001 C CNN
+	1    8650 700
+	0    -1   -1   0
+$EndComp
+$Comp
+L Connector:Screw_Terminal_01x02 J1
+U 1 1 5C34BA95
+P 6750 700
+F 0 "J1" V 6716 512 50  0000 R CNN
+F 1 "Screw_Terminal_01x02" V 6625 512 50  0000 R CNN
+F 2 "TerminalBlock:TerminalBlock_bornier-2_P5.08mm" H 6750 700 50  0001 C CNN
+F 3 "~" H 6750 700 50  0001 C CNN
+	1    6750 700
+	0    -1   -1   0
+$EndComp
+Text GLabel 6750 950  3    50   Input ~ 0
+12v
+Text GLabel 6850 950  3    50   Input ~ 0
+GND
+Wire Wire Line
+	6750 900  6750 950
+Wire Wire Line
+	6850 900  6850 950
+Text GLabel 8050 900  3    50   Input ~ 0
+OUT1+
+Text GLabel 8150 900  3    50   Input ~ 0
+OUT1-
+Text GLabel 8650 900  3    50   Input ~ 0
+OUT2+
+Text GLabel 8750 900  3    50   Input ~ 0
+OUT2-
+Text GLabel 7300 900  3    50   Input ~ 0
+TXD
+Text GLabel 7400 900  3    50   Input ~ 0
+RXD
+Text GLabel 7500 900  3    50   Input ~ 0
+GND
+$Comp
+L power:+12V #PWR?
+U 1 1 5C36ECC0
+P 1000 800
+F 0 "#PWR?" H 1000 650 50  0001 C CNN
+F 1 "+12V" H 1015 973 50  0000 C CNN
+F 2 "" H 1000 800 50  0001 C CNN
+F 3 "" H 1000 800 50  0001 C CNN
+	1    1000 800
+	1    0    0    -1
+$EndComp
+Wire Wire Line
+	1000 800  1000 1250
 $EndSCHEMATC

Commit message: PWM2
Parts:
- C1: footprint Capacitor_THT:CP_Radial_D4.0mm_P2.00mm -> Capacitor_THT:C_Disc_D7.5mm_W2.5mm_P5.00mm
- C2: footprint Capacitor_THT:C_Disc_D3.0mm_W1.6mm_P2.50mm -> Capacitor_THT:CP_Radial_D5.0mm_P2.50mm
- J2: footprint Connector_PinHeader_1.00mm:PinHeader_1x03_P1.00mm_Vertical -> Connector_PinHeader_2.54mm:PinHeader_1x03_P2.54mm_Horizontal
- Q1, Q2, Q4, Q5: footprint Package_TO_SOT_THT:TO-92_Inline -> Package_TO_SOT_THT:TO-92_Inline_Wide
- R10, R5, R6, R7, R8, R9: footprint Resistor_THT:R_Axial_DIN0207_L6.3mm_D2.5mm_P2.54mm_Vertical -> Resistor_THT:R_Axial_DIN0204_L3.6mm_D1.6mm_P7.62mm_Horizontal
- R4: footprint Resistor_THT:R_Axial_DIN0207_L6.3mm_D2.5mm_P2.54mm_Vertical -> Resistor_THT:R_Axial_DIN0207_L6.3mm_D2.5mm_P7.62mm_Horizontal
Connections:
- net OUT2-: now also J4.1 (Pin_1); no longer J4.2 (Pin_2)
- net +12V renamed 12v
- net 12v: now also J4.2 (Pin_2); no longer J4.1 (Pin_1)
Changed lines of the file:
@@
 F 0 "Q1" H 8891 2596 50  0000 L CNN
 F 1 "2N3904" H 8891 2505 50  0000 L CNN
-F 2 "Package_TO_SOT_THT:TO-92_Inline" H 8900 2475 50  0001 L CIN
+F 2 "Package_TO_SOT_THT:TO-92_Inline_Wide" H 8900 2475 50  0001 L CIN
 F 3 "https://www.fairchildsemi.com/datasheets/2N/2N3904.pdf" H 8700 2550 50  0001 L CNN
 	1    8700 2550
@@
 F 0 "Q2" H 9391 3146 50  0000 L CNN
 F 1 "2N3904" H 9391 3055 50  0000 L CNN
-F 2 "Package_TO_SOT_THT:TO-92_Inline" H 9400 3025 50  0001 L CIN
+F 2 "Package_TO_SOT_THT:TO-92_Inline_Wide" H 9400 3025 50  0001 L CIN
 F 3 "https://www.fairchildsemi.com/datasheets/2N/2N3904.pdf" H 9200 3100 50  0001 L CNN
 	1    9200 3100
@@
 F 0 "R6" H 8870 1996 50  0000 L CNN
 F 1 "1k" H 8870 1905 50  0000 L CNN
-F 2 "Resistor_THT:R_Axial_DIN0207_L6.3mm_D2.5mm_P2.54mm_Vertical" V 8730 1950 50  0001 C CNN
+F 2 "Resistor_THT:R_Axial_DIN0204_L3.6mm_D1.6mm_P7.62mm_Horizontal" V 8730 1950 50  0001 C CNN
 F 3 "~" H 8800 1950 50  0001 C CNN
 	1    8800 1950
@@
 F 0 "R7" H 9320 1996 50  0000 L CNN
 F 1 "500" H 9320 1905 50  0000 L CNN
-F 2 "Resistor_THT:R_Axial_DIN0207_L6.3mm_D2.5mm_P2.54mm_Vertical" V 9180 1950 50  0001 C CNN
+F 2 "Resistor_THT:R_Axial_DIN0204_L3.6mm_D1.6mm_P7.62mm_Horizontal" V 9180 1950 50  0001 C CNN
 F 3 "~" H 9250 1950 50  0001 C CNN
 	1    9250 1950
@@
 F 0 "R5" V 7843 2550 50  0000 C CNN
 F 1 "200" V 7934 2550 50  0000 C CNN
-F 2 "Resistor_THT:R_Axial_DIN0207_L6.3mm_D2.5mm_P2.54mm_Vertical" V 7980 2550 50  0001 C CNN
+F 2 "Resistor_THT:R_Axial_DIN0204_L3.6mm_D1.6mm_P7.62mm_Horizontal" V 7980 2550 50  0001 C CNN
 F 3 "~" H 8050 2550 50  0001 C CNN
 	1    8050 2550
@@
 F 0 "R4" H 4670 3546 50  0000 L CNN
 F 1 "100k" H 4670 3455 50  0000 L CNN
-F 2 "Resistor_THT:R_Axial_DIN0207_L6.3mm_D2.5mm_P2.54mm_Vertical" V 4530 3500 50  0001 C CNN
+F 2 "Resistor_THT:R_Axial_DIN0207_L6.3mm_D2.5mm_P7.62mm_Horizontal" V 4530 3500 50  0001 C CNN
 F 3 "~" H 4600 3500 50  0001 C CNN
 	1    4600 3500
@@
 F 0 "Q4" H 8891 4746 50  0000 L CNN
 F 1 "2N3904" H 8891 4655 50  0000 L CNN
-F 2 "Package_TO_SOT_THT:TO-92_Inline" H 8900 4625 50  0001 L CIN
+F 2 "Package_TO_SOT_THT:TO-92_Inline_Wide" H 8900 4625 50  0001 L CIN
 F 3 "https://www.fairchildsemi.com/datasheets/2N/2N3904.pdf" H 8700 4700 50  0001 L CNN
 	1    8700 4700
@@
 F 0 "Q5" H 9391 5296 50  0000 L CNN
 F 1 "2N3904" H 9391 5205 50  0000 L CNN
-F 2 "Package_TO_SOT_THT:TO-92_Inline" H 9400 5175 50  0001 L CIN
+F 2 "Package_TO_SOT_THT:TO-92_Inline_Wide" H 9400 5175 50  0001 L CIN
 F 3 "https://www.fairchildsemi.com/datasheets/2N/2N3904.pdf" H 9200 5250 50  0001 L CNN
 	1    9200 5250
@@
 F 0 "R9" H 8870 4146 50  0000 L CNN
 F 1 "1k" H 8870 4055 50  0000 L CNN
-F 2 "Resistor_THT:R_Axial_DIN0207_L6.3mm_D2.5mm_P2.54mm_Vertical" V 8730 4100 50  0001 C CNN
+F 2 "Resistor_THT:R_Axial_DIN0204_L3.6mm_D1.6mm_P7.62mm_Horizontal" V 8730 4100 50  0001 C CNN
 F 3 "~" H 8800 4100 50  0001 C CNN
 	1    8800 4100
@@
 F 0 "R10" H 9320 4146 50  0000 L CNN
 F 1 "500" H 9320 4055 50  0000 L CNN
-F 2 "Resistor_THT:R_Axial_DIN0207_L6.3mm_D2.5mm_P2.54mm_Vertical" V 9180 4100 50  0001 C CNN
+F 2 "Resistor_THT:R_Axial_DIN0204_L3.6mm_D1.6mm_P7.62mm_Horizontal" V 9180 4100 50  0001 C CNN
 F 3 "~" H 9250 4100 50  0001 C CNN
 	1    9250 4100
@@
 F 0 "R8" V 7843 4700 50  0000 C CNN
 F 1 "200" V 7934 4700 50  0000 C CNN
-F 2 "Resistor_THT:R_Axial_DIN0207_L6.3mm_D2.5mm_P2.54mm_Vertical" V 7980 4700 50  0001 C CNN
+F 2 "Resistor_THT:R_Axial_DIN0204_L3.6mm_D1.6mm_P7.62mm_Horizontal" V 7980 4700 50  0001 C CNN
 F 3 "~" H 8050 4700 50  0001 C CNN
 	1    8050 4700
@@
 F 0 "C2" H 1968 1696 50  0000 L CNN
 F 1 "100u" H 1968 1605 50  0000 L CNN
-F 2 "Capacitor_THT:C_Disc_D3.0mm_W1.6mm_P2.50mm" H 1888 1500 50  0001 C CNN
+F 2 "Capacitor_THT:CP_Radial_D5.0mm_P2.50mm" H 1888 1500 50  0001 C CNN
 F 3 "~" H 1850 1650 50  0001 C CNN
 	1    1850 1650
@@
 F 0 "C1" H 1115 1596 50  0000 L CNN
 F 1 "100n" H 1115 1505 50  0000 L CNN
-F 2 "Capacitor_THT:CP_Radial_D4.0mm_P2.00mm" H 1038 1400 50  0001 C CNN
+F 2 "Capacitor_THT:C_Disc_D7.5mm_W2.5mm_P5.00mm" H 1038 1400 50  0001 C CNN
 F 3 "~" H 1000 1550 50  0001 C CNN
 	1    1000 1550
@@
 F 0 "J2" V 7460 840 50  0000 L CNN
 F 1 "Conn_01x03_Male" V 7551 840 50  0000 L CNN
-F 2 "Connector_PinHeader_1.00mm:PinHeader_1x03_P1.00mm_Vertical" H 7400 700 50  0001 C CNN
+F 2 "Connector_PinHeader_2.54mm:PinHeader_1x03_P2.54mm_Horizontal" H 7400 700 50  0001 C CNN
 F 3 "~" H 7400 700 50  0001 C CNN
 	1    7400 700
@@
 Text GLabel 8150 900  3    50   Input ~ 0
 OUT1-
+Text GLabel 8750 900  3    50   Input ~ 0
+OUT2+
 Text GLabel 8650 900  3    50   Input ~ 0
-OUT2+
-Text GLabel 8750 900  3    50   Input ~ 0
 OUT2-
 Text GLabel 7300 900  3    50   Input ~ 0
@@
 Text GLabel 7500 900  3    50   Input ~ 0
 GND
-$Comp
-L power:+12V #PWR?
-U 1 1 5C36ECC0
-P 1000 800
-F 0 "#PWR?" H 1000 650 50  0001 C CNN
-F 1 "+12V" H 1015 973 50  0000 C CNN
-F 2 "" H 1000 800 50  0001 C CNN
-F 3 "" H 1000 800 50  0001 C CNN
-	1    1000 800
-	1    0    0    -1
-$EndComp
-Wire Wire Line
-	1000 800  1000 1250
 $EndSCHEMATC
