File: pwm-3/esp-pwm/esp-pwm.sch (KiCad schematic (older format))
At the start: 31 parts, among them J1 Screw_Terminal_01x02, J2 Screw_Terminal_01x02, J3 Screw_Terminal_01x02, J4 Screw_Terminal_01x02, J5 Screw_Terminal_01x02, Q1 2N3904, Q10 IRF540N, Q11 IRF540N, Q12 IRF540N, Q2 2N3904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

Commit message: ...
Parts:
- removed J1, J2, J3, J4, J5: Screw_Terminal_01x02, TerminalBlock:TerminalBlock_bornier-2_P5.08mm, symbol Connector:Screw_Terminal_01x02
- removed Q1, Q2, Q4, Q5, Q6, Q7, Q8, Q9: 2N3904, Package_TO_SOT_THT:TO-92, symbol Transistor_BJT:2N3904
- removed Q10, Q11, Q12, Q3: IRF540N, Package_TO_SOT_THT:TO-220-3_Vertical, symbol Transistor_FET:IRF540N
- removed R1, R4, R5, R6: 200, Resistor_THT:R_Axial_DIN0516_L15.5mm_D5.0mm_P20.32mm_Horizontal, symbol Device:R
- removed R10, R11, R12, R3: 500, Resistor_THT:R_Axial_DIN0516_L15.5mm_D5.0mm_P20.32mm_Horizontal, symbol Device:R
- removed R2, R7, R8, R9: 1K, Resistor_THT:R_Axial_DIN0516_L15.5mm_D5.0mm_P20.32mm_Horizontal, symbol Device:R
- removed U2: WeMos_mini, wemos_mini_d1:D1_mini_board, symbol wemos_mini_d1:WeMos_mini
- added C1, C2: 100n, Capacitor_THT:C_Axial_L3.8mm_D2.6mm_P7.50mm_Horizontal, symbol Device:C
- added J6: Screw_Terminal_01x04, Connector_PinHeader_2.54mm:PinHeader_1x04_P2.54mm_Horizontal, symbol Connector:Screw_Terminal_01x04
- added U2: NodeMCU1.0(ESP-12E), ESP8266:NodeMCU1.0(12-E), symbol ESP8266:NodeMCU1.0(ESP-12E)
Connections:
- net labels added: 12v, 5v, Ctrl, Radio
- net labels removed: 12V, 5V, CTRL1, CTRL2, CTRL3, CTRL4, OUT1+, OUT1-, OUT2+, OUT2-, OUT3+, OUT3-, OUT4+, OUT4-
- wire segments 108 -> 19
