File: pwm-driver/pwm-driver/pwm-driver.kicad_pcb (KiCad board)
At the start: 2 copper layers, 10 parts, among them J1 12V, J2 GND, J4 CTRL, J5 OUT, Q1 2N3904, Q2 2N3904, Q3 IRF540N

Commit message: ...
Parts:
- Q1, Q2: footprint Package_TO_SOT_THT:TO-92_Inline -> Package_TO_SOT_THT:TO-92_Inline_Wide
- moved Q2 4.58 mm to (129.5, 71.1), turned to 90 degrees
- moved R2 2.93 mm to (124.5, 76.2)
- moved R3 2.54 mm to (114.3, 81.3)
- moved R1 1.27 mm to (119.4, 76.2)
Routing:
- net Net-(Q1-Pad3): track 22.8 -> 17.8 mm
- net Net-(Q2-Pad3): track 58.4 -> 54.9 mm
- net Net-(Q1-Pad2): track 7.62 -> 10.4 mm
- net GND: track 38.1 -> 36.8 mm
- net 12v: track 14.0 -> 15.2 mm

Commit message: ...
Parts:
- moved J2 30.2 mm to (125.7, 62.2)
- moved J5 28.5 mm to (125.7, 66.0)
- moved J4 20.9 mm to (125.7, 69.8)
- moved J1 18.8 mm to (125.7, 73.7)
- moved Q2 17.6 mm to (114.3, 62.2), turned to 270 degrees
- moved R2 12.8 mm to (111.8, 74.9)
- moved Q3 10.9 mm to (108.0, 71.1), turned to 90 degrees
- moved Q1 9.25 mm to (119.4, 62.2), turned to 270 degrees
- moved R1 6.84 mm to (121.9, 69.8)
- moved R3 6.84 mm to (116.8, 74.9)
Routing:
- net Net-(Q2-Pad3): track 54.9 -> 14.0 mm
- net Out: track 0.00 -> 35.6 mm
- net GND: track 36.8 -> 21.6 mm
- net Ctrl: track 0.00 -> 8.89 mm
- net Net-(Q1-Pad2): track 10.4 -> 7.62 mm
- net 12v: track 15.2 -> 17.8 mm
- net Net-(Q1-Pad3): track 17.8 -> 15.2 mm
